File: CAD/Eagle/HFT-Core-Module_1V0.sch (EAGLE design)
At the start: 394 parts, among them Q0521 ABS07-32.768KHZ, Q0811 ABM03B-32.000MHZ, Q0911 ABM3B-16MHZ-10-R50-1-U, T1201 MMBT2222, T1202 MMBT2222, T1203 MMBT2222, U0111 STM32L4Z_144PIN_SMPS, U0431 PAM2305AAB120, U0601 LM4120IM5-3.0, U0611 MAX5217, U0631 CFPT-141-20MHZ, U0641 OPA354, U0701 Si5338, U0801 SX1276, U0901 AX5243, U0911 PE4259, U0921 PE4259, U0991 PE4259, U1011 MAX5136AGTG+, U1101 MCP3911A0-E-SS, U1121 OPA354, U1131 OPA354, U1141 OPA354, U1201 NHD-C0220BIZ_2X20CHARS, U1301 MPU-9250, U1311 MS5607-02BA03, U1321 SHT31-DIS, U1401 SOLARPANEL_3V3_5MA1_25MM_X_20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, U1402 SPV1040T, U1501 TS5A23166, U1601 PAM2305AAB330, U1701 TS5A23166, U1801 TS5A23166, U1901 TS5A23166, X1261 TTE_EN11-HSM, X2101 SMA_SMT_AMPHENOL-901-143, X2111 SMA_SMT_AMPHENOL-901-143, X2201 CUI SJ1-3535NS, X2211 CUI SJ1-3535NS, X2311 2X20/90_1MM27_HARWIN_M50-3202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, X2312 2X20/90_1MM27_HARWIN_M50-3202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, X2321 2X20/90_1MM27_HARWIN_M50-3202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, X2322 2X20/90_1MM27_HARWIN_M50-3202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, X2331 2X20/90_1MM27_HARWIN_M50-3202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, X2332 2X20/90_1MM27_HARWIN_M50-3202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

Commit message: HW_1V0 - it is getting more delicate now
Changed lines of the file:
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@@
 </segment>
 </bus>
-<bus name="PA[8..15]">
+<bus name="PA[8..10],PA_USB_N,PA_USB_P,PA[13..15]">
 <segment>
 <wire x1="147.32" y1="172.72" x2="238.76" y2="172.72" width="0.762" layer="92"/>
@@
 </instances>
 <busses>
-<bus name="GND,+3V3,+5V0,CLK0P,CLK0N,CLK1P,CLK1N,CLK2P,CLK2N,MCU_WAKEUP,MCU_I2C1_SCL,MCU_I2C1_SDA,MCU_I2C2_SCL,MCU_I2C2_SDA,MCU_I2C3_SCL,MCU_I2C3_SDA,MCU_SPI1_SCK,MCU_SPI1_MOSI,MCU_SPI1_MISO,I2S_SCK_OUT,I2S_SD_OUT,I2S_MCLK_OUT,I2S_FS_OUT,PA[0..15],PB[0..15],PC[0..15],PD[0..15],PE[0..15],PF[0..15],PG[0..15],PH[0..3]">
+<bus name="GND,+3V3,+5V0,CLK0_P,CLK0_N,CLK1_P,CLK1_N,CLK2_P,CLK2_N,MCU_WAKEUP,MCU_I2C1_SCL,MCU_I2C1_SDA,MCU_I2C2_SCL,MCU_I2C2_SDA,MCU_I2C3_SCL,MCU_I2C3_SDA,MCU_SPI1_SCK,MCU_SPI1_MOSI,MCU_SPI1_MISO,I2S_SCK_OUT,I2S_SD_OUT,I2S_MCLK_OUT,I2S_FS_OUT,PA[0..15],PB[0..15],PC[0..15],PD[0..15],PE[0..15],PF[0..15],PG[0..15],PH[0..3]">
 <segment>
 <wire x1="246.38" y1="132.08" x2="246.38" y2="83.82" width="0.762" layer="92"/>
