File: CAD/Eagle/HFT-Core-Module_1V0.brd (EAGLE design)
At the start: 96.5 x 96.5 mm, 402 parts, among them Q0521 ABS07-32.768KHZ, Q0811 ABM03B-32.000MHZ, Q0911 ABM3B-16MHZ-10-R50-1-U, T1201 MMBT2222, T1202 MMBT2222, T1203 MMBT2222, U0111 STM32L4Z_144PIN_SMPS, U0431 PAM2305AAB120, U0601 LM4120IM5-3.0, U0611 MAX5217, U0631 CFPT-141-20MHZ, U0641 OPA354, U0701 Si5338, U0801 SX1276, U0901 AX5243, U0911 PE4259, U0921 PE4259, U0991 PE4259, U1101 MCP3911A0-E-SS, U1111 MAX5136AGTG+, U1121 OPA354, U1131 OPA354, U1141 OPA354, U1201 NHD-C0220BIZ_2X20CHARS, U1301 MPU-9250, U1311 MS5607-02BA03, U1321 SHT31-DIS, U1401 SOLARPANEL_3V3_5MA1_25MM_X_20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, U1402 SPV1040T, U1501 TS5A23166, U1601 SC189ZSKTRT, U1701 TS5A23166, U1801 TS5A23166, U1901 TS5A23166, X1261 TTE_EN11-HSM, X2001 MOLEX 105017-0001, X2101 SMA_SMT_AMPHENOL-901-143, SAM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, X2111 SMA_SMT_AMPHENOL-901-143, SAM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, X2201 CUI SJ1-3535NS, X2211 CUI SJ1-3535NS, X2311 2X20/90_1MM27_HARWIN_M50-3202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, X2312 2X20/90_1MM27_HARWIN_M50-3202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, X2321 2X20/90_1MM27_HARWIN_M50-3202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, X2322 2X20/90_1MM27_HARWIN_M50-3202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, X2331 2X20/90_1MM27_HARWIN_M50-3202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, X2332 2X20/90_1MM27_HARWIN_M50-3202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

Commit message: HW_1V0 - SWD header, XO 32.768kHz caps, RESET resistor removed
Parts:
- C0511: value 1.5pF -> 22pF
- R0311: value 3.3kR -> N/A
Changed lines of the file:
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@@
 <attribute name="VALUE" x="45.085" y="57.785" size="0.6096" layer="27" font="vector" ratio="10" rot="R270"/>
 </element>
-<element name="R0311" library="rcl" package="R0603" value="3.3kR" x="45.085" y="57.15" smashed="yes" rot="R90">
+<element name="R0311" library="rcl" package="R0603" value="N/A" x="45.085" y="57.15" smashed="yes" rot="R90">
 <attribute name="NAME" x="44.7675" y="59.055" size="0.6096" layer="25" font="vector" ratio="10" rot="R90"/>
 <attribute name="VALUE" x="46.99" y="56.515" size="0.6096" layer="27" font="vector" ratio="10" rot="R90"/>
@@
 <attribute name="VALUE" x="48.775" y="65.93" size="0.6096" layer="27" font="vector" ratio="10"/>
 </element>
-<element name="C0511" library="rcl" package="C0603" value="1.5pF" x="48.26" y="71.12" smashed="yes" rot="R180">
+<element name="C0511" library="rcl" package="C0603" value="22pF" x="48.26" y="71.12" smashed="yes" rot="R180">
 <attribute name="NAME" x="46.99" y="72.0725" size="0.6096" layer="25" font="vector" ratio="10"/>
 <attribute name="VALUE" x="48.895" y="73.025" size="0.6096" layer="27" font="vector" ratio="10" rot="R180"/>

Commit message: HW_1V0 - LCD-backlight resistors changed
Parts:
- R1201: value 1.8kR -> 2.0kR
- R1202: value 5.2kR -> 1.5kR
- R1203: value 68R -> 27R
- R1204, R1207: value 2.2kR -> 2.0kR
- R1205, R1208: value 1.8kR -> 1.5kR
- R1206, R1209: value 10R -> 27R
Changed lines of the file:
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@@
 <attribute name="VALUE" x="20.32" y="17.145" size="0.6096" layer="28" font="vector" ratio="10" rot="MR270"/>
 </element>
-<element name="R1209" library="rcl" package="R0805" value="10R" x="21.59" y="14.605" smashed="yes" rot="MR0">
+<element name="R1209" library="rcl" package="R0805" value="27R" x="21.59" y="14.605" smashed="yes" rot="MR0">
 <attribute name="NAME" x="26.035" y="14.2875" size="0.6096" layer="26" font="vector" ratio="10" rot="MR0"/>
 <attribute name="VALUE" x="22.225" y="12.065" size="0.6096" layer="28" font="vector" ratio="10" rot="MR0"/>
 </element>
-<element name="R1208" library="rcl" package="R0603" value="1.8kR" x="21.59" y="16.51" smashed="yes" rot="MR0">
+<element name="R1208" library="rcl" package="R0603" value="1.5kR" x="21.59" y="16.51" smashed="yes" rot="MR0">
 <attribute name="NAME" x="26.035" y="16.1925" size="0.6096" layer="26" font="vector" ratio="10" rot="MR0"/>
 <attribute name="VALUE" x="22.225" y="14.605" size="0.6096" layer="28" font="vector" ratio="10" rot="MR0"/>
 </element>
-<element name="R1207" library="rcl" package="R0603" value="2.2kR" x="62.23" y="47.625" smashed="yes" rot="MR90">
+<element name="R1207" library="rcl" package="R0603" value="2.0kR" x="62.23" y="47.625" smashed="yes" rot="MR90">
 <attribute name="NAME" x="61.9125" y="43.18" size="0.6096" layer="26" font="vector" ratio="10" rot="MR90"/>
 <attribute name="VALUE" x="60.325" y="46.99" size="0.6096" layer="28" font="vector" ratio="10" rot="MR90"/>
 </element>
-<element name="R1206" library="rcl" package="R0805" value="10R" x="21.59" y="18.415" smashed="yes" rot="MR0">
+<element name="R1206" library="rcl" package="R0805" value="27R" x="21.59" y="18.415" smashed="yes" rot="MR0">
 <attribute name="NAME" x="26.035" y="18.0975" size="0.6096" layer="26" font="vector" ratio="10" rot="MR0"/>
 <attribute name="VALUE" x="22.225" y="15.875" size="0.6096" layer="28" font="vector" ratio="10" rot="MR0"/>
 </element>
-<element name="R1203" library="rcl" package="R0805" value="68R" x="21.59" y="22.225" smashed="yes" rot="MR0">
+<element name="R1203" library="rcl" package="R0805" value="27R" x="21.59" y="22.225" smashed="yes" rot="MR0">
 <attribute name="NAME" x="26.035" y="21.9075" size="0.6096" layer="26" font="vector" ratio="10" rot="MR0"/>
 <attribute name="VALUE" x="22.225" y="19.685" size="0.6096" layer="28" font="vector" ratio="10" rot="MR0"/>
 </element>
-<element name="R1205" library="rcl" package="R0603" value="1.8kR" x="21.59" y="20.32" smashed="yes" rot="MR0">
+<element name="R1205" library="rcl" package="R0603" value="1.5kR" x="21.59" y="20.32" smashed="yes" rot="MR0">
 <attribute name="NAME" x="26.035" y="20.0025" size="0.6096" layer="26" font="vector" ratio="10" rot="MR0"/>
 <attribute name="VALUE" x="22.225" y="18.415" size="0.6096" layer="28" font="vector" ratio="10" rot="MR0"/>
 </element>
-<element name="R1202" library="rcl" package="R0603" value="5.2kR" x="21.59" y="24.13" smashed="yes" rot="MR0">
+<element name="R1202" library="rcl" package="R0603" value="1.5kR" x="21.59" y="24.13" smashed="yes" rot="MR0">
 <attribute name="NAME" x="26.035" y="24.13" size="0.6096" layer="26" font="vector" ratio="10" rot="MR0"/>
 <attribute name="VALUE" x="22.225" y="22.225" size="0.6096" layer="28" font="vector" ratio="10" rot="MR0"/>
 </element>
-<element name="R1204" library="rcl" package="R0603" value="2.2kR" x="59.055" y="47.625" smashed="yes" rot="R90">
+<element name="R1204" library="rcl" package="R0603" value="2.0kR" x="59.055" y="47.625" smashed="yes" rot="R90">
 <attribute name="NAME" x="59.055" y="43.18" size="0.6096" layer="25" font="vector" ratio="10" rot="R90"/>
 <attribute name="VALUE" x="60.96" y="46.99" size="0.6096" layer="27" font="vector" ratio="10" rot="R90"/>
 </element>
-<element name="R1201" library="rcl" package="R0603" value="1.8kR" x="80.645" y="65.405" smashed="yes" rot="MR0">
+<element name="R1201" library="rcl" package="R0603" value="2.0kR" x="80.645" y="65.405" smashed="yes" rot="MR0">
 <attribute name="NAME" x="79.0575" y="65.0875" size="0.6096" layer="26" font="vector" ratio="10" rot="MR0"/>
 <attribute name="VALUE" x="81.28" y="63.5" size="0.6096" layer="28" font="vector" ratio="10" rot="MR0"/>

Commit message: HW_1V0 - I2C R values and addresses changed
Parts:
- R1331, R1332: value 3.9kR -> 1.0kR
Changed lines of the file:
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@@
 <attribute name="VALUE" x="43.18" y="26.67" size="0.6096" layer="28" font="vector" ratio="10" rot="MR90"/>
 </element>
-<element name="R1331" library="rcl" package="R0603" value="3.9kR" x="5.715" y="15.875" smashed="yes" rot="MR0">
+<element name="R1331" library="rcl" package="R0603" value="1.0kR" x="5.715" y="15.875" smashed="yes" rot="MR0">
 <attribute name="NAME" x="10.16" y="15.5575" size="0.6096" layer="26" font="vector" ratio="10" rot="MR0"/>
 <attribute name="VALUE" x="6.35" y="13.97" size="0.6096" layer="28" font="vector" ratio="10" rot="MR0"/>
 </element>
-<element name="R1332" library="rcl" package="R0603" value="3.9kR" x="5.715" y="13.335" smashed="yes" rot="MR0">
+<element name="R1332" library="rcl" package="R0603" value="1.0kR" x="5.715" y="13.335" smashed="yes" rot="MR0">
 <attribute name="NAME" x="10.16" y="13.0175" size="0.6096" layer="26" font="vector" ratio="10" rot="MR0"/>
 <attribute name="VALUE" x="6.35" y="11.43" size="0.6096" layer="28" font="vector" ratio="10" rot="MR0"/>

Commit message: HW_1V0 - Solar DC/DC needs 100uF at the input, MCU runs 24MHz and emits 12MHz for the Si5338
Parts:
- C1401: value 10uF -> 100uF
Changed lines of the file:
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@@
 <attribute name="VALUE" x="23.495" y="36.195" size="0.6096" layer="28" font="vector" ratio="10" rot="MR180"/>
 </element>
-<element name="C1401" library="rcl" package="C0805" value="10uF" x="19.05" y="44.45" smashed="yes" rot="MR90">
+<element name="C1401" library="rcl" package="C0805" value="100uF" x="19.05" y="44.45" smashed="yes" rot="MR90">
 <attribute name="NAME" x="20.32" y="43.18" size="0.6096" layer="26" font="vector" ratio="10" rot="MR90"/>
 <attribute name="VALUE" x="16.51" y="43.18" size="0.6096" layer="28" font="vector" ratio="10" rot="MR90"/>

Commit message: HW_1V0 - SX1276 change of cap to 12pF
Parts:
- C0812: value 4.7p -> 12pF
Changed lines of the file:
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@@
 <attribute name="VALUE" x="62.23" y="14.605" size="0.6096" layer="28" font="vector" ratio="10" rot="MR270"/>
 </element>
-<element name="C0812" library="rcl" package="C0603" value="4.7p" x="69.215" y="10.795" smashed="yes" rot="MR270">
+<element name="C0812" library="rcl" package="C0603" value="12pF" x="69.215" y="10.795" smashed="yes" rot="MR270">
 <attribute name="NAME" x="67.945" y="9.525" size="0.6096" layer="26" font="vector" ratio="10" rot="MR90"/>
 <attribute name="VALUE" x="71.12" y="11.43" size="0.6096" layer="28" font="vector" ratio="10" rot="MR270"/>

Commit message: HW_1V0 - ADC resistor values changed, ADC OSC2 should be connected to GND (reminder added)
Parts:
- R1132, R1135, R1142, R1145: value 33kR -> 10MR
Changed lines of the file:
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@@
 <layers>
 <layer number="1" name="Top" color="4" fill="1" visible="yes" active="yes"/>
-<layer number="2" name="Layer_2" color="1" fill="3" visible="yes" active="yes"/>
+<layer number="2" name="Layer_2" color="1" fill="3" visible="no" active="yes"/>
 <layer number="3" name="Route3" color="4" fill="3" visible="no" active="no"/>
 <layer number="4" name="Route4" color="1" fill="4" visible="no" active="no"/>
@@
 <layer number="13" name="Route13" color="4" fill="5" visible="no" active="no"/>
 <layer number="14" name="Route14" color="1" fill="6" visible="no" active="no"/>
-<layer number="15" name="Layer_15" color="4" fill="6" visible="yes" active="yes"/>
+<layer number="15" name="Layer_15" color="4" fill="6" visible="no" active="yes"/>
 <layer number="16" name="Bottom" color="1" fill="1" visible="yes" active="yes"/>
 <layer number="17" name="Pads" color="2" fill="1" visible="yes" active="yes"/>
@@
 <layer number="19" name="Unrouted" color="6" fill="1" visible="yes" active="yes"/>
 <layer number="20" name="Dimension" color="5" fill="1" visible="yes" active="yes"/>
-<layer number="21" name="tPlace" color="7" fill="1" visible="yes" active="yes"/>
+<layer number="21" name="tPlace" color="7" fill="1" visible="no" active="yes"/>
 <layer number="22" name="bPlace" color="7" fill="1" visible="yes" active="yes"/>
-<layer number="23" name="tOrigins" color="15" fill="1" visible="yes" active="yes"/>
+<layer number="23" name="tOrigins" color="15" fill="1" visible="no" active="yes"/>
 <layer number="24" name="bOrigins" color="15" fill="1" visible="yes" active="yes"/>
-<layer number="25" name="tNames" color="7" fill="1" visible="yes" active="yes"/>
+<layer number="25" name="tNames" color="7" fill="1" visible="no" active="yes"/>
 <layer number="26" name="bNames" color="7" fill="1" visible="yes" active="yes"/>
 <layer number="27" name="tValues" color="7" fill="1" visible="no" active="yes"/>
 <layer number="28" name="bValues" color="7" fill="1" visible="no" active="yes"/>
-<layer number="29" name="tStop" color="7" fill="3" visible="yes" active="yes"/>
+<layer number="29" name="tStop" color="7" fill="3" visible="no" active="yes"/>
 <layer number="30" name="bStop" color="7" fill="6" visible="yes" active="yes"/>
 <layer number="31" name="tCream" color="7" fill="4" visible="no" active="yes"/>
@@
 <layer number="42" name="bRestrict" color="1" fill="10" visible="no" active="yes"/>
 <layer number="43" name="vRestrict" color="2" fill="10" visible="no" active="yes"/>
-<layer number="44" name="Drills" color="7" fill="1" visible="yes" active="yes"/>
-<layer number="45" name="Holes" color="7" fill="1" visible="yes" active="yes"/>
+<layer number="44" name="Drills" color="7" fill="1" visible="no" active="yes"/>
+<layer number="45" name="Holes" color="7" fill="1" visible="no" active="yes"/>
 <layer number="46" name="Milling" color="3" fill="1" visible="no" active="yes"/>
-<layer number="47" name="Measures" color="13" fill="1" visible="yes" active="yes"/>
-<layer number="48" name="Document" color="7" fill="1" visible="yes" active="yes"/>
-<layer number="49" name="Reference" color="7" fill="1" visible="yes" active="yes"/>
+<layer number="47" name="Measures" color="13" fill="1" visible="no" active="yes"/>
+<layer number="48" name="Document" color="7" fill="1" visible="no" active="yes"/>
+<layer number="49" name="Reference" color="7" fill="1" visible="no" active="yes"/>
 <layer number="50" name="dxf" color="7" fill="1" visible="no" active="no"/>
-<layer number="51" name="tDocu" color="7" fill="1" visible="yes" active="yes"/>
+<layer number="51" name="tDocu" color="7" fill="1" visible="no" active="yes"/>
 <layer number="52" name="bDocu" color="15" fill="1" visible="yes" active="yes"/>
 <layer number="53" name="tGND_GNDA" color="7" fill="9" visible="no" active="no"/>
@@
 <attribute name="VALUE" x="71.91375" y="81.43875" size="0.6096" layer="28" font="vector" ratio="10" rot="MR180"/>
 </element>
-<element name="R1132" library="rcl" package="R0603" value="33kR" x="85.725" y="73.66" smashed="yes" rot="MR180">
+<element name="R1132" library="rcl" package="R0603" value="10MR" x="85.725" y="73.66" smashed="yes" rot="MR180">
 <attribute name="NAME" x="86.995" y="72.39" size="0.6096" layer="26" font="vector" ratio="10" rot="MR0"/>
 <attribute name="VALUE" x="85.09" y="75.565" size="0.6096" layer="28" font="vector" ratio="10" rot="MR180"/>
 </element>
-<element name="R1142" library="rcl" package="R0603" value="33kR" x="87.63" y="66.04" smashed="yes" rot="MR180">
+<element name="R1142" library="rcl" package="R0603" value="10MR" x="87.63" y="66.04" smashed="yes" rot="MR180">
 <attribute name="NAME" x="88.9" y="64.4525" size="0.6096" layer="26" font="vector" ratio="10" rot="MR0"/>
 <attribute name="VALUE" x="86.995" y="67.945" size="0.6096" layer="28" font="vector" ratio="10" rot="MR180"/>
@@
 <attribute name="VALUE" x="87.15375" y="77.47" size="0.6096" layer="28" font="vector" ratio="10" rot="MR180"/>
 </element>
-<element name="R1135" library="rcl" package="R0603" value="33kR" x="87.78875" y="76.835" smashed="yes" rot="MR180">
+<element name="R1135" library="rcl" package="R0603" value="10MR" x="87.78875" y="76.835" smashed="yes" rot="MR180">
 <attribute name="NAME" x="89.05875" y="77.7875" size="0.6096" layer="26" font="vector" ratio="10" rot="MR0"/>
 <attribute name="VALUE" x="87.15375" y="78.74" size="0.6096" layer="28" font="vector" ratio="10" rot="MR180"/>
 </element>
-<element name="R1145" library="rcl" package="R0603" value="33kR" x="91.44" y="67.945" smashed="yes" rot="MR0">
+<element name="R1145" library="rcl" package="R0603" value="10MR" x="91.44" y="67.945" smashed="yes" rot="MR0">
 <attribute name="NAME" x="92.71" y="66.3575" size="0.6096" layer="26" font="vector" ratio="10" rot="MR0"/>
 <attribute name="VALUE" x="92.075" y="66.04" size="0.6096" layer="28" font="vector" ratio="10" rot="MR0"/>

Commit message: HW_1V0 - CAD/Eagle - AX5243 clock out is 8MHz
Connections:
- net AX_16MHZ renamed AX_8MHZ
Changed lines of the file:
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@@
 <wire x1="68.8975" y1="29.425" x2="68.58" y2="29.1075" width="0.2032" layer="16" curve="-90"/>
 </signal>
-<signal name="AX_16MHZ">
+<signal name="AX_8MHZ">
 <contactref element="R1021" pad="2"/>
 <contactref element="R0714" pad="1"/>
