File: CAD/Eagle/HFT-Core-Module_1V1.sch (EAGLE design)
At the start: 406 parts, among them Q0521 ABS07-32.768KHZ, Q0811 ABM03B-32.000MHZ, Q0911 ABM3B-16MHZ-10-R50-1-U, T1201 MMBT2222, T1202 MMBT2222, T1203 MMBT2222, U0001 PAM2305AAB120, U0111 STM32L4Z_144PIN_SMPS, U0601 LM4120IM5-3.0, U0611 MAX5217, U0631 CFPT-141-20MHZ, U0641 OPA354, U0701 Si5338, U0801 SX1276, U0901 AX5243, U0911 PE4259, U0921 PE4259, U0991 PE4259, U1101 MCP3911A0-E-SS, U1111 MAX5136AGTG+, U1131 OPA354, U1141 OPA354, U1201 NHD-C0220BIZ_2X20CHARS, U1301 MPU-9250, U1311 MS5607-02BA03, U1321 SHT31-DIS, U1402 SPV1040T, U1501 TS5A23166, U1601 SC189ZSKTRT, U1701 TS5A23166, U1801 TS5A23166, U1901 TS5A23166, X1261 TTE_EN11-HSM, X1401 WIRE-TO-BOARD_5MM08_1X02, X2001 MOLEX 105017-0001, X2101 SMA_SMT_AMPHENOL-901-143, SAM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, X2111 SMA_SMT_AMPHENOL-901-143, SAM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, X2201 CUI SJ1-3535NS, X2211 CUI SJ1-3535NS, X2311 2X20/90_1MM27_HARWIN_M50-3202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, X2312 2X20/90_1MM27_HARWIN_M50-3202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, X2321 2X20/90_1MM27_HARWIN_M50-3202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, X2322 2X20/90_1MM27_HARWIN_M50-3202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, X2331 2X20/90_1MM27_HARWIN_M50-3202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, X2332 2X20/90_1MM27_HARWIN_M50-3202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

Commit message: HW_1V1 - CAD/Eagle - re-arangement of pages done
Parts:
- removed C1111, C1112, C1301, C1303, C1321: 100nF, rcl:C-EUC0603
- removed C1113: 47pF, rcl:C-EUC0603
- removed C1128, C1129: 100nF, df4iah_rcl:C-EUC0603
- removed C1131, C1141: 220nF, df4iah_rcl:C-EUC0603
- removed C1132, C1142: 100uF, df4iah_rcl:C-EUC0805
- removed C1302: 10nF, rcl:C-EUC0603
- removed D0451: CMAD6001, df4iah_diode:D_SOD923
- removed L1112: 10uH, rcl:L-EUL2012C
- removed R0261, R0262, R0263, R1107, R1108, R1109, R1114: 47R, rcl:R-EU_R0603
- removed R1104, R1105: 22kR, rcl:R-EU_R0603
- removed R1110: 33kR, rcl:R-EU_R0603
- removed R1131, R1141: 10kR, rcl:R-EU_R0603
- removed R1132, R1135, R1142, R1145: 10MR, rcl:R-EU_R0603
- removed R1301: 68R, rcl:R-EU_R0603
- removed R1331, R1332: 1.0kR, rcl:R-EU_R0603
- removed U0801: SX1276, df4iah_rf:SX1276
- removed U0911, U0921: PE4259, df4iah_rf:PE4259
- removed U1101: MCP3911A0-E-SS, df4iah_adc:MCP3911
- removed U1111: MAX5136AGTG+, df4iah_dac:MAX5136
- removed U1131, U1141: OPA354, df4iah_opamp:OPA354
- removed U1301: MPU-9250, df4iah_sensors:MPU-9250
- removed U1311: MS5607-02BA03, df4iah_sensors:MS5607-02BA03
- removed U1321: SHT31-DIS, df4iah_sensors:SHT31-DIS
- added C0004, C0012: 1uF, rcl:C-EUC0603
- added C0005, C0009: 2.7nF, df4iah_rcl:C-EUC0603
- added C0006, C0013: 4.7uF, rcl:C-EUC0603
- added C0011, C0015: 100nF, rcl:C-EUC0603
- added C0014: 10uF, rcl:C-EUC0603
- added C0016, C0018: 2.2uF, rcl:C-EUC0603
- added C0019, C0020: 10nF, df4iah_rcl:C-EUC0603
- added L0002: 10uH, df4iah_rcl:R-EU_R0603
- added R0005, R0006: 1.0kR, rcl:R-EU_R0603
- added R0007, R0029, R0030, R0031, R0032, R0033, R0034, R0035: 47R, rcl:R-EU_R0603
- added R0011, R0012: 560R, rcl:R-EU_R0603
- added R0015: 68R, rcl:R-EU_R0603
- added R0016, R0017: 100R, rcl:R-EU_R0603
- added R0018, R0019, R0020, R0021, R0022, R0023, R0028: D.C., rcl:R-EU_R0603
- added R0026, R0027: 10kR, rcl:R-EU_R0603
- added U0002: PCM1863, df4iah_adc:PCM1863
- added U0005: (no value), df4iah_dac:WM8523
- C0531: value TZY2Z100AC01R00 -> JR200
- C0532: value 12pF -> 8.2pF
- C1102: value 100nF -> 10uF
- C1104, C1105: value 220nF -> 10uF
- L1102: device rcl:L-EUL2012C -> df4iah_rcl:R-EU_R0603
- R0321: value 10kR -> 33kR
Connections:
- net +3V3_20MHZ renamed +3V3_XO
- removed net AUDIO_OUT_L_OP: C1132.1, U1131.-IN, U1131.OUT
- removed net AUDIO_OUT_R_OP: C1142.1, U1141.-IN, U1141.OUT
- removed net MAX5136_!READY: R1114.2, U1111.!READY
- removed net MAX5136_AVDD: C1112.2, L1112.1, U1111.AVDD, U1111.M/!Z
- removed net MAX5136_OUT0: R1131.1, U1111.OUT0
- removed net MAX5136_OUT0_R: C1131.1, R1131.2
- removed net MAX5136_OUT0_SUM: C1131.2, R1132.2, R1135.2, U1131.+IN
- removed net MAX5136_OUT1: R1141.1, U1111.OUT1
- removed net MAX5136_OUT1_R: C1141.1, R1141.2
- removed net MAX5136_OUT1_SUM: C1141.2, R1142.2, R1145.2, U1141.+IN
- removed net MAX5136_REF: C1113.1, R1132.1, R1142.1, U1111.REFI, U1111.REFO
- removed net MCP3911_!DR: R1106.1, U1101.!DR
- removed net MCP3911_CH0+: C1104.2, R1104.2, U1101.CH0+
- removed net MCP3911_CH1+: C1105.2, R1105.2, U1101.CH1+
- removed net MCP3911_MDAT0: R1108.1, U1101.MDAT0
- removed net MCP3911_MDAT1: R1109.1, U1101.MDAT1
- removed net MCP3911_REFINOUT: C1103.2, U1101.REFINOUT
- removed net MCP3911_SDO: R1107.1, U1101.SDO
- removed net MCU_OUT_AUDIO_ADC_NRESET: R0261.2, R1110.2, U1101.!RESET
- removed net MCU_OUT_AUDIO_ADC_SEL: R0262.2, U1101.!CS
- removed net MCU_OUT_AUDIO_DAC_SEL: R0263.2, U1111.!CS
- removed net MPU_INT: R1301.1, U1301.INT
- removed net MPU_REGOUT: C1303.1, U1301.REGOUT
- removed net MVP3911_AVDD: C1102.2, L1102.1, U1101.AVDD
- new net AUDIOADC_AVDD: C1103.2, L1102.1, U0002.AVDD
- new net AUDIOADC_BCK: R0030.1, U0002.BCK
- new net AUDIOADC_DOUT: R0029.1, U0002.DOUT
- new net AUDIOADC_INTA: R1106.1, U0002.GPIO1/INTA/DMIN
- new net AUDIOADC_LDO: C0014.1, C0015.1, U0002.LDO
- new net AUDIOADC_LRCK: R0031.1, U0002.LRCK
- new net AUDIOADC_MIC_BIAS: R0028.2, U0002.MIC_BIAS
- new net AUDIOADC_VINL1: C0019.1, R0016.2, U0002.VINL1/VIN1P
- new net AUDIOADC_VINL1_R: C1104.2, R0016.1
- new net AUDIOADC_VINL2: R0018.2, U0002.VINL2/VIN1M
- new net AUDIOADC_VINL3: R0019.2, U0002.VINL3/VIN4P
- new net AUDIOADC_VINL4: R0020.2, U0002.VINL4/VIN4M
- new net AUDIOADC_VINR1: C0020.1, R0017.2, U0002.VINR1/VIN2P
- new net AUDIOADC_VINR1_R: C1105.2, R0017.1
- new net AUDIOADC_VINR2: R0021.2, U0002.VINR2/VIN2M
- new net AUDIOADC_VINR3: R0022.2, U0002.VINR3/VIN3P
- new net AUDIOADC_VINR4: R0023.2, U0002.VINR4/VIN3M
- new net AUDIOADC_VREF: C0018.1, U0002.VREF
- new net AUDIO_DAC_AVDD: C0006.2, L0002.1, U0005.AVDD
- new net AUDIO_DAC_BCLK: R0032.2, U0005.BCLK
- new net AUDIO_DAC_CPCA: C0004.1, U0005.CPCA
- new net AUDIO_DAC_CPCB: C0004.2, U0005.CPCB
- new net AUDIO_DAC_CPVOUTN: C0012.2, U0005.CPVOUTN
- new net AUDIO_DAC_DACDAT: R0007.2, U0005.DACDAT
- new net AUDIO_DAC_LINEVOUTL: R0011.1, U0005.LINEVOUTL
- new net AUDIO_DAC_LINEVOUTR: R0012.1, U0005.LINEVOUTR
- new net AUDIO_DAC_LRCLK: R0033.2, U0005.LRCLK
- new net AUDIO_DAC_MCLK: R0034.2, U0005.MCLK
- new net AUDIO_DAC_VMID: C0016.2, U0005.VMID
- new net AUDIO_DAC_ZFLAG: R0035.1, U0005.ZFLAG
- new net N$3: C1101.2
- net +3V3: now also C0011.1, R0005.2, R0006.2; no longer C1301.1, C1302.1, C1321.1, D0451.A, R1331.2, R1332.2, U0801.VBAT_ANA, U0801.VBAT_DIG, U0801.VBAT_RF, U0911.VDD_!CTRL, U0921.VDD_!CTRL, U1301.!CS, U1301.VDD, U1301.VDDIO, U1311.CSB_!ADDR, U1311.PS, U1311.VDD, U1321.!RESET, U1321.VDD
- net +3V3_HICUR: now also C0013.1, C1102.1, L0002.2, U0002.DVDD, U0002.IOVDD, U0005.LINEVDD; no longer C1111.1, C1128.1, C1129.1, L1112.2, U1101.DVDD, U1111.!LDAC, U1111.DVDD, U1131.V+, U1141.V+
- net AUDIO_IN_L: now also R0026.2
- net AUDIO_IN_R: now also R0027.2
- net AUDIO_OUT_L: now also C0009.1, R0011.2; no longer C1132.2
- net AUDIO_OUT_R: now also C0005.1, R0012.2; no longer C1142.2
- net GND: now also C0005.2, C0006.1, C0009.2, C0011.2, C0012.1, C0013.2, C0014.2, C0015.2, C0016.1, C0018.2, C0019.2, C0020.2, C1102.2, R0026.1, R0027.1, U0002.AGND, U0002.DGND, U0002.MD0, U0002.MS/AD, U0005.!CS!/!MUTE, U0005.AGND, U0005.CIFMODE, U0005.LINEGND, U0005.SDOUT/DEEMPH; no longer C1101.2, C1102.1, C1111.2, C1112.1, C1113.2, C1128.2, C1129.2, C1301.2, C1302.2, C1303.2, C1321.2, R1104.1, R1105.1, R1110.1, R1135.1, R1145.1, U0801.GND@15, U0801.GND@23, U0801.GND@26, U0801.GND@PAD, U0911.GND, U0921.GND, U1101.AGND, U1101.CH0-, U1101.CH1-, U1101.DGND, U1101.OSC2, U1101.REFIN-, U1111.GND, U1131.V-, U1141.V-, U1301.AD0/SDO, U1301.FSYNC, U1301.GND, U1311.GND, U1321.ADDR, U1321.PAD, U1321.R, U1321.VSS
- net MCU_I2C4_SCL: now also R0006.1, U0002.MC/SCL, U0005.SCLK/AIFMODE1; no longer R1332.1, U1301.SCL/SCLK, U1311.SCL_SCLK, U1321.SCL
- net MCU_I2C4_SDA: now also R0005.1, U0002.MOSI/SDA, U0005.SDA/AIFMODE0; no longer R1331.1, U1301.SDA/SDI, U1311.SDI_SDA, U1321.SDA
- net MCU_OUT_SX_SEL: no longer U0801.NSS
- net MCU_SPI3_MOSI: no longer U0801.MOSI, U1101.SDI, U1111.DIN
- net MCU_SPI3_SCK: no longer U1101.SCK, U1111.SCLK
- net MCU_VBAT: no longer D0451.C
- net PA15: now also R0035.2
- net PB13: now also R0030.2
- net PC11: no longer R1107.2
- net PC8: no longer R1114.1
- net PC9: no longer R0263.1
- net PD0: no longer R1109.2
- net PD1: no longer R1108.2
- net PD11: now also R0029.2
- net PD12: now also R0031.2
- net PD3: no longer R0261.1
- net PD5: no longer R0262.1
- net PE10: now also R0034.1
- net PE3: now also R0007.1
- net PE8: now also R0032.1
- net PE9: now also R0033.1
- net PF13: now also R0015.2; no longer R1301.2
- net SI5338_CLK3B_2: now also U0002.SCKI; no longer U1101.OSC1
- net SX_DIO0: no longer U0801.DIO0
- net SX_DIO1: no longer U0801.DIO1
- net SX_DIO2: no longer U0801.DIO2
- net SX_DIO3: no longer U0801.DIO3
- net SX_DIO4: no longer U0801.DIO4
- net SX_DIO5: no longer U0801.DIO5
- net SX_HF_1: no longer U0911.RFC
- net SX_LF_1: no longer U0921.RFC
- net SX_MISO: no longer U0801.MISO
- net SX_NRESET: no longer U0801.!RESET
- net SX_RFI_HF: no longer U0801.RFI_HF
- net SX_RFI_HF_5: no longer U0911.RF2
- net SX_RFI_LF: no longer U0801.RFI_LF
- net SX_RFI_LF_5: no longer U0921.RF2
- net SX_RFO_HF: no longer U0801.RFO_HF
- net SX_RFO_HF_4: no longer U0911.RF1
- net SX_RFO_LF: no longer U0801.RFO_LF
- net SX_RFO_LF_5: no longer U0921.RF1
- net SX_RXTX: no longer U0801.RXTX/RFMOD
- net SX_TX_!RX!_CTRL: no longer U0911.CTRL, U0921.CTRL
- net SX_VR_ANA: no longer U0801.VR_ANA
- net SX_VR_DIG: no longer U0801.VR_DIG
- net SX_VR_PA: no longer U0801.VR_PA
- net SX_XTA: no longer U0801.XTA
- net SX_XTB: no longer U0801.XTB
Other:
- note added: "16x2 char LCD Rotary encoder"
- note added: "4p5F..20pF"
- note added: "9-axis sensor: BNO-085 SPI"
- note added: "A0"
- note added: "A1"
- note added: "AX5243 UHF TRX (ch2)"
- note added: "Add EEPROM: CAT24C64"
- note added: "Climate sensor"
- note added: "Climate sensor: BME680 I2C addr: 0x76"
- note added: "Crystal 32.768 kHz"
- note added: "D.C."
- note added: "EEPROM: I2C addr: 0x50"
- note added: "Electronic switch for USB-Power <--> 5V"
- note added: "I2C EEPROM 8k x 8Bit"
- note added: "I2C address space: Addr Device 0x0C (9axis Mag) 0x1A Audio DAC 0x38 TCXO DAC 0x3D LCD 0x4A Audio ADC 0x50 EEPROM 0x68 (9axis Gyro/Accel) 0x70 Si5338 PLL 0x76 Weather sensor"
- note added: "I2S audio ADC"
- note added: "I2S audio DAC"
- note added: "I2S audio stereo A/D-Converter I2C addr: 0x4A"
- note added: "I2S audio stereo D/A-Converter I2C addr: 0x1A"
- note added: "I2S1B_FS_OUT"
- note added: "I2S1B_MCLK_OUT"
- note added: "I2S1B_SCK_OUT"
- note added: "I2S1B_SD_OUT"
- note added: "Load: 10kR"
- note added: "MCU: LSE 32.768 kHz"
- note added: "MCU_AUDIO_DAC_ZFLAG_IN"
- note added: "MCU_I2S2A_FS_IN"
- note added: "MCU_I2S2A_SCK_IN"
- note added: "MCU_I2S2A_SD_IN"
- note added: "MCU_IN_AUDIO_ADC_INT"
- note added: "PMIC 3.3V --> 1.2V"
- note added: "PMIC 5V --> 3.3V"
- note added: "Position tracking"
- note added: "SX1262 UHF TRX (ch1)"
- note added: "SX1262 antenna SW"
- note added: "Si5338 PLL"
- note added: "Solar power harvesting"
- note added: "VCTCXO 20MHz (XO)"
- note added: "VHF / UHF SX1262 - channel 1 SPI"
- note removed: "3..10pF"
- note removed: "9-axis sensor: MPU-9250 I2C addr: 0x68 / 0x0C"
- note removed: "Add QUADSPI EEPROM"
- note removed: "Audio stereo A/D-Converter SPI"
- note removed: "Audio stereo D/A-Converter SPI"
- note removed: "Baro sensor: MS5607-02BA03 I2C addr: 0x76"
- note removed: "Change to 0603"
- note removed: "Electronic switch for USB <--> 5V"
- note removed: "MCU LF Osc"
- note removed: "MCU switchboard"
- note removed: "MCU: low frequency oscillator"
- note removed: "MCU_IN_AUDIO_ADC_MDAT0"
- note removed: "MCU_IN_AUDIO_ADC_MDAT1"
- note removed: "MCU_IN_AUDIO_ADC_NDR"
- note removed: "MCU_IN_AUDIO_DAC_NRDY"
- note removed: "RH sensor: Sensirion SHT3x I2C addr: 0x44"
- note removed: "TODO: To be replaced by ICM-20948 (1.8 Volt !) Use SPI instead of I2C and Level Converter"
- note removed: "To be replaced by I2S components."
- note removed: "VCTCXO 20MHz"
- note removed: "VHF / UHF SX1276 - channel 1 SPI"
- note removed: "not needed!"
